Commit message: R2D2 Example

File: src/assignment4/urdf/lynxmotion.urdf.xacro (robot description, xacro)
@@ -1,10 +1,215 @@
 <?xml version="1.0"?>
-<robot name="lynxmotion">
-	<link name="base_link">
-		<visual>
-			<geometry>
-				<cylinder length="0.6" radius="0.2"/>
-			</geometry>
-		</visual>
-	</link>
+<robot name="macroed" xmlns:xacro="http://ros.org/wiki/xacro">
+  <xacro:property name="width" value="0.2" />
+  <xacro:property name="leglen" value="0.6" />
+  <xacro:property name="polelen" value="0.2" />
+  <xacro:property name="bodylen" value="0.6" />
+  <xacro:property name="baselen" value="0.4" />
+  <xacro:property name="wheeldiam" value="0.07" />
+  <xacro:property name="pi" value="3.1415" />
+  <material name="blue">
+    <color rgba="0 0 0.8 1"/>
+  </material>
+  <material name="black">
+    <color rgba="0 0 0 1"/>
+  </material>
+  <material name="white">
+    <color rgba="1 1 1 1"/>
+  </material>
+  <xacro:macro name="default_inertial" params="mass">
+    <inertial>
+      <mass value="${mass}" />
+      <inertia ixx="1.0" ixy="0.0" ixz="0.0" iyy="1.0" iyz="0.0" izz="1.0" />
+    </inertial>
+  </xacro:macro>
+  <link name="base_link">
+    <visual>
+      <geometry>
+        <cylinder radius="${width}" length="${bodylen}"/>
+      </geometry>
+      <material name="blue"/>
+    </visual>
+    <collision>
+      <geometry>
+        <cylinder radius="${width}" length="${bodylen}"/>
+      </geometry>
+    </collision>
+    <xacro:default_inertial mass="10"/>
+  </link>
+  <xacro:macro name="wheel" params="prefix suffix reflect">
+    <link name="${prefix}_${suffix}_wheel">
+      <visual>
+        <origin xyz="0 0 0" rpy="${pi/2} 0 0" />
+        <geometry>
+          <cylinder radius="${wheeldiam/2}" length="0.1"/>
+        </geometry>
+        <material name="black"/>
+      </visual>
+      <collision>
+        <origin xyz="0 0 0" rpy="${pi/2} 0 0" />
+        <geometry>
+          <cylinder radius="${wheeldiam/2}" length="0.1"/>
+        </geometry>
+      </collision>
+      <xacro:default_inertial mass="1"/>
+    </link>
+    <joint name="${prefix}_${suffix}_wheel_joint" type="continuous">
+      <axis xyz="0 1 0" rpy="0 0 0" />
+      <parent link="${prefix}_base"/>
+      <child link="${prefix}_${suffix}_wheel"/>
+      <origin xyz="${baselen*reflect/3} 0 -${wheeldiam/2+.05}" rpy="0 0 0"/>
+    </joint>
+  </xacro:macro>
+  <xacro:macro name="leg" params="prefix reflect">
+    <link name="${prefix}_leg">
+      <visual>
+        <geometry>
+          <box size="${leglen} 0.1 0.2"/>
+        </geometry>
+        <origin xyz="0 0 -${leglen/2}" rpy="0 ${pi/2} 0"/>
+        <material name="white"/>
+      </visual>
+      <collision>
+        <geometry>
+          <box size="${leglen} 0.1 0.2"/>
+        </geometry>
+        <origin xyz="0 0 -${leglen/2}" rpy="0 ${pi/2} 0"/>
+      </collision>
+      <xacro:default_inertial mass="10"/>
+    </link>
+    <joint name="base_to_${prefix}_leg" type="fixed">
+      <parent link="base_link"/>
+      <child link="${prefix}_leg"/>
+      <origin xyz="0 ${reflect*(width+.02)} 0.25" />
+    </joint>
+    <link name="${prefix}_base">
+      <visual>
+        <geometry>
+          <box size="${baselen} 0.1 0.1"/>
+        </geometry>
+        <material name="white"/>
+      </visual>
+      <collision>
+        <geometry>
+          <box size="${baselen} 0.1 0.1"/>
+        </geometry>
+      </collision>
+      <xacro:default_inertial mass="10"/>
+    </link>
+    <joint name="${prefix}_base_joint" type="fixed">
+      <parent link="${prefix}_leg"/>
+      <child link="${prefix}_base"/>
+      <origin xyz="0 0 ${-leglen}" />
+    </joint>
+    <xacro:wheel prefix="${prefix}" suffix="front" reflect="1"/>
+    <xacro:wheel prefix="${prefix}" suffix="back" reflect="-1"/>
+  </xacro:macro>
+  <xacro:leg prefix="right" reflect="-1" />
+  <xacro:leg prefix="left" reflect="1" />
+  <joint name="gripper_extension" type="prismatic">
+    <parent link="base_link"/>
+    <child link="gripper_pole"/>
+    <limit effort="1000.0" lower="-${width*2-.02}" upper="0" velocity="0.5"/>
+    <origin rpy="0 0 0" xyz="${width-.01} 0 0.2"/>
+  </joint>
+  <link name="gripper_pole">
+    <visual>
+      <geometry>
+        <cylinder length="${polelen}" radius="0.01"/>
+      </geometry>
+      <origin xyz="${polelen/2} 0 0" rpy="0 ${pi/2} 0 "/>
+    </visual>
+    <collision>
+      <geometry>
+        <cylinder length="${polelen}" radius="0.01"/>
+      </geometry>
+      <origin xyz="${polelen/2} 0 0" rpy="0 ${pi/2} 0 "/>
+    </collision>
+    <xacro:default_inertial mass="0.05"/>
+  </link>
+  <xacro:macro name="gripper" params="prefix reflect">
+    <joint name="${prefix}_gripper_joint" type="revolute">
+      <axis xyz="0 0 ${reflect}"/>
+      <limit effort="1000.0" lower="0.0" upper="0.548" velocity="0.5"/>
+      <origin rpy="0 0 0" xyz="${polelen} ${reflect*0.01} 0"/>
+      <parent link="gripper_pole"/>
+      <child link="${prefix}_gripper"/>
+    </joint>
+    <link name="${prefix}_gripper">
+      <visual>
+        <origin rpy="${(reflect-1)/2*pi} 0 0" xyz="0 0 0"/>
+        <geometry>
+          <mesh filename="package://urdf_tutorial/meshes/l_finger.dae"/>
+        </geometry>
+      </visual>
+      <collision>
+        <geometry>
+          <mesh filename="package://urdf_tutorial/meshes/l_finger.dae"/>
+        </geometry>
+        <origin rpy="${(reflect-1)/2*pi} 0 0" xyz="0 0 0"/>
+      </collision>
+      <xacro:default_inertial mass="0.05"/>
+    </link>
+    <joint name="${prefix}_tip_joint" type="fixed">
+      <parent link="${prefix}_gripper"/>
+      <child link="${prefix}_tip"/>
+    </joint>
+    <link name="${prefix}_tip">
+      <visual>
+        <origin rpy="${(reflect-1)/2*pi} 0 0" xyz="0.09137 0.00495 0"/>
+        <geometry>
+          <mesh filename="package://urdf_tutorial/meshes/l_finger_tip.dae"/>
+        </geometry>
+      </visual>
+      <collision>
+        <geometry>
+          <mesh filename="package://urdf_tutorial/meshes/l_finger_tip.dae"/>
+        </geometry>
+        <origin rpy="${(reflect-1)/2*pi} 0 0" xyz="0.09137 0.00495 0"/>
+      </collision>
+      <xacro:default_inertial mass="0.05"/>
+    </link>
+  </xacro:macro>
+  <xacro:gripper prefix="left" reflect="1" />
+  <xacro:gripper prefix="right" reflect="-1" />
+  <link name="head">
+    <visual>
+      <geometry>
+        <sphere radius="${width}"/>
+      </geometry>
+      <material name="white"/>
+    </visual>
+    <collision>
+      <geometry>
+        <sphere radius="${width}"/>
+      </geometry>
+    </collision>
+    <xacro:default_inertial mass="2"/>
+  </link>
+  <joint name="head_swivel" type="continuous">
+    <parent link="base_link"/>
+    <child link="head"/>
+    <axis xyz="0 0 1"/>
+    <origin xyz="0 0 ${bodylen/2}"/>
+  </joint>
+  <link name="box">
+    <visual>
+      <geometry>
+        <box size="0.08 0.08 0.08"/>
+      </geometry>
+      <material name="blue"/>
+      <origin xyz="-0.04 0 0"/>
+    </visual>
+    <collision>
+      <geometry>
+        <box size="0.08 0.08 0.08"/>
+      </geometry>
+    </collision>
+    <xacro:default_inertial mass="1"/>
+  </link>
+  <joint name="tobox" type="fixed">
+    <parent link="head"/>
+    <child link="box"/>
+    <origin xyz="${.707*width+0.04} 0 ${.707*width}"/>
+  </joint>
 </robot>

Commit message: Iets met armen

File: src/assignment4/urdf/lynxmotion.urdf.xacro (robot description, xacro)
@@ -1,215 +1,80 @@
 <?xml version="1.0"?>
 <robot name="macroed" xmlns:xacro="http://ros.org/wiki/xacro">
-  <xacro:property name="width" value="0.2" />
-  <xacro:property name="leglen" value="0.6" />
-  <xacro:property name="polelen" value="0.2" />
-  <xacro:property name="bodylen" value="0.6" />
-  <xacro:property name="baselen" value="0.4" />
-  <xacro:property name="wheeldiam" value="0.07" />
-  <xacro:property name="pi" value="3.1415" />
-  <material name="blue">
-    <color rgba="0 0 0.8 1"/>
-  </material>
-  <material name="black">
-    <color rgba="0 0 0 1"/>
-  </material>
-  <material name="white">
-    <color rgba="1 1 1 1"/>
-  </material>
-  <xacro:macro name="default_inertial" params="mass">
-    <inertial>
-      <mass value="${mass}" />
-      <inertia ixx="1.0" ixy="0.0" ixz="0.0" iyy="1.0" iyz="0.0" izz="1.0" />
-    </inertial>
-  </xacro:macro>
+  <xacro:property name="M_PI" value="3.14159"/>
+  <xacro:property name="base_width" value="0.069" />
+  <xacro:property name="base_height" value="0.069" />
+  <xacro:property name="servo_width" value="0.020" />
+  <xacro:property name="servo_length" value="0.040" />
+  <xacro:property name="shoulder_height" value="0.010" />
+  <xacro:property name="shoulder_offset" value="0.015" />
+  <xacro:property name="upperarm_length" value="0.127" />
+  <xacro:property name="hand_length" value="0.086" />
+  <!-- Links -->
   <link name="base_link">
     <visual>
+      <origin xyz="0 0 ${base_height/2}" rpy="0 0 0"/>
       <geometry>
-        <cylinder radius="${width}" length="${bodylen}"/>
+        <cylinder radius="${base_width}" length="${base_height}"/>
       </geometry>
-      <material name="blue"/>
     </visual>
-    <collision>
+  </link>
+  <link name="shoulder_rotate_link">
+    <visual>
+      <origin xyz="0 0 0" rpy="0 0 0"/>
       <geometry>
-        <cylinder radius="${width}" length="${bodylen}"/>
+        <cylinder radius="${base_width}" length="${shoulder_height}"/>
       </geometry>
-    </collision>
-    <xacro:default_inertial mass="10"/>
+    </visual>
   </link>
-  <xacro:macro name="wheel" params="prefix suffix reflect">
-    <link name="${prefix}_${suffix}_wheel">
-      <visual>
-        <origin xyz="0 0 0" rpy="${pi/2} 0 0" />
-        <geometry>
-          <cylinder radius="${wheeldiam/2}" length="0.1"/>
-        </geometry>
-        <material name="black"/>
-      </visual>
-      <collision>
-        <origin xyz="0 0 0" rpy="${pi/2} 0 0" />
-        <geometry>
-          <cylinder radius="${wheeldiam/2}" length="0.1"/>
-        </geometry>
-      </collision>
-      <xacro:default_inertial mass="1"/>
-    </link>
-    <joint name="${prefix}_${suffix}_wheel_joint" type="continuous">
-      <axis xyz="0 1 0" rpy="0 0 0" />
-      <parent link="${prefix}_base"/>
-      <child link="${prefix}_${suffix}_wheel"/>
-      <origin xyz="${baselen*reflect/3} 0 -${wheeldiam/2+.05}" rpy="0 0 0"/>
-    </joint>
-  </xacro:macro>
-  <xacro:macro name="leg" params="prefix reflect">
-    <link name="${prefix}_leg">
-      <visual>
-        <geometry>
-          <box size="${leglen} 0.1 0.2"/>
-        </geometry>
-        <origin xyz="0 0 -${leglen/2}" rpy="0 ${pi/2} 0"/>
-        <material name="white"/>
-      </visual>
-      <collision>
-        <geometry>
-          <box size="${leglen} 0.1 0.2"/>
-        </geometry>
-        <origin xyz="0 0 -${leglen/2}" rpy="0 ${pi/2} 0"/>
-      </collision>
-      <xacro:default_inertial mass="10"/>
-    </link>
-    <joint name="base_to_${prefix}_leg" type="fixed">
-      <parent link="base_link"/>
-      <child link="${prefix}_leg"/>
-      <origin xyz="0 ${reflect*(width+.02)} 0.25" />
-    </joint>
-    <link name="${prefix}_base">
-      <visual>
-        <geometry>
-          <box size="${baselen} 0.1 0.1"/>
-        </geometry>
-        <material name="white"/>
-      </visual>
-      <collision>
-        <geometry>
-          <box size="${baselen} 0.1 0.1"/>
-        </geometry>
-      </collision>
-      <xacro:default_inertial mass="10"/>
-    </link>
-    <joint name="${prefix}_base_joint" type="fixed">
-      <parent link="${prefix}_leg"/>
-      <child link="${prefix}_base"/>
-      <origin xyz="0 0 ${-leglen}" />
-    </joint>
-    <xacro:wheel prefix="${prefix}" suffix="front" reflect="1"/>
-    <xacro:wheel prefix="${prefix}" suffix="back" reflect="-1"/>
-  </xacro:macro>
-  <xacro:leg prefix="right" reflect="-1" />
-  <xacro:leg prefix="left" reflect="1" />
-  <joint name="gripper_extension" type="prismatic">
+  <link name="shoulder_updown_link">
+    <visual>
+      <origin xyz="0 0 0" rpy="0 0 0"/>
+      <geometry>
+        <cylinder radius="${servo_width}" length="${servo_length}"/>
+      </geometry>
+    </visual>
+  </link>
+  <link name="upperarm_link">
+    <visual>
+      <origin xyz="0 0 0" rpy="0 0 0"/>
+      <geometry>
+        <box size="${upperarm_length} ${servo_width} ${servo_width}"/>
+      </geometry>
+    </visual>
+  </link>
+  <!-- <link name="elbow_link">
+    <visual>
+      <origin xyz="0 0 0" rpy="0 0 0"/>
+      <geometry>
+        <cylinder radius="${servo_width}" length="${servo_length}"/>
+      </geometry>
+    </visual>
+  </link> -->
+  <!-- Joints -->
+  <joint name="shoulder_rotate_joint" type="revolute">
+    <origin xyz="0 0 ${base_height + shoulder_height}" rpy="0 0 0"/>
     <parent link="base_link"/>
-    <child link="gripper_pole"/>
-    <limit effort="1000.0" lower="-${width*2-.02}" upper="0" velocity="0.5"/>
-    <origin rpy="0 0 0" xyz="${width-.01} 0 0.2"/>
+    <child link="shoulder_rotate_link"/>
+    <axis xyz="0 0 1"/>
+    <limit lower="-${M_PI/2}" upper="${M_PI/2}" effort="0" velocity="3.67"/>
   </joint>
-  <link name="gripper_pole">
-    <visual>
-      <geometry>
-        <cylinder length="${polelen}" radius="0.01"/>
-      </geometry>
-      <origin xyz="${polelen/2} 0 0" rpy="0 ${pi/2} 0 "/>
-    </visual>
-    <collision>
-      <geometry>
-        <cylinder length="${polelen}" radius="0.01"/>
-      </geometry>
-      <origin xyz="${polelen/2} 0 0" rpy="0 ${pi/2} 0 "/>
-    </collision>
-    <xacro:default_inertial mass="0.05"/>
-  </link>
-  <xacro:macro name="gripper" params="prefix reflect">
-    <joint name="${prefix}_gripper_joint" type="revolute">
-      <axis xyz="0 0 ${reflect}"/>
-      <limit effort="1000.0" lower="0.0" upper="0.548" velocity="0.5"/>
-      <origin rpy="0 0 0" xyz="${polelen} ${reflect*0.01} 0"/>
-      <parent link="gripper_pole"/>
-      <child link="${prefix}_gripper"/>
-    </joint>
-    <link name="${prefix}_gripper">
-      <visual>
-        <origin rpy="${(reflect-1)/2*pi} 0 0" xyz="0 0 0"/>
-        <geometry>
-          <mesh filename="package://urdf_tutorial/meshes/l_finger.dae"/>
-        </geometry>
-      </visual>
-      <collision>
-        <geometry>
-          <mesh filename="package://urdf_tutorial/meshes/l_finger.dae"/>
-        </geometry>
-        <origin rpy="${(reflect-1)/2*pi} 0 0" xyz="0 0 0"/>
-      </collision>
-      <xacro:default_inertial mass="0.05"/>
-    </link>
-    <joint name="${prefix}_tip_joint" type="fixed">
-      <parent link="${prefix}_gripper"/>
-      <child link="${prefix}_tip"/>
-    </joint>
-    <link name="${prefix}_tip">
-      <visual>
-        <origin rpy="${(reflect-1)/2*pi} 0 0" xyz="0.09137 0.00495 0"/>
-        <geometry>
-          <mesh filename="package://urdf_tutorial/meshes/l_finger_tip.dae"/>
-        </geometry>
-      </visual>
-      <collision>
-        <geometry>
-          <mesh filename="package://urdf_tutorial/meshes/l_finger_tip.dae"/>
-        </geometry>
-        <origin rpy="${(reflect-1)/2*pi} 0 0" xyz="0.09137 0.00495 0"/>
-      </collision>
-      <xacro:default_inertial mass="0.05"/>
-    </link>
-  </xacro:macro>
-  <xacro:gripper prefix="left" reflect="1" />
-  <xacro:gripper prefix="right" reflect="-1" />
-  <link name="head">
-    <visual>
-      <geometry>
-        <sphere radius="${width}"/>
-      </geometry>
-      <material name="white"/>
-    </visual>
-    <collision>
-      <geometry>
-        <sphere radius="${width}"/>
-      </geometry>
-    </collision>
-    <xacro:default_inertial mass="2"/>
-  </link>
-  <joint name="head_swivel" type="continuous">
-    <parent link="base_link"/>
-    <child link="head"/>
+  <joint name="shoulder_updown_joint" type="revolute">
+    <origin xyz="0 0 ${shoulder_offset}" rpy="${M_PI/2} 0 0"/>
+    <parent link="shoulder_rotate_link"/>
+    <child link="shoulder_updown_link"/>
     <axis xyz="0 0 1"/>
-    <origin xyz="0 0 ${bodylen/2}"/>
+    <limit lower="0" upper="${M_PI}" effort="0" velocity="3.67"/>
   </joint>
-  <link name="box">
-    <visual>
-      <geometry>
-        <box size="0.08 0.08 0.08"/>
-      </geometry>
-      <material name="blue"/>
-      <origin xyz="-0.04 0 0"/>
-    </visual>
-    <collision>
-      <geometry>
-        <box size="0.08 0.08 0.08"/>
-      </geometry>
-    </collision>
-    <xacro:default_inertial mass="1"/>
-  </link>
-  <joint name="tobox" type="fixed">
-    <parent link="head"/>
-    <child link="box"/>
-    <origin xyz="${.707*width+0.04} 0 ${.707*width}"/>
+  <joint name="upperarm_joint" type="fixed">
+    <origin xyz="${upperarm_length/2} 0 0" rpy="${M_PI/2} 0 0"/>
+    <parent link="shoulder_updown_link"/>
+    <child link="upperarm_link"/>
   </joint>
+  <!-- <joint name="elbow_joint" type="revolute">
+    <origin xyz="0 0 0" rpy="${M_PI/2} 0 0"/>
+    <parent link="upperarm_link"/>
+    <child link="elbow_link"/>
+    <axis xyz="0 0 1"/>
+    <limit lower="-${M_PI/2}" upper="${M_PI/2}" effort="0" velocity="3.67"/>
+  </joint> -->
 </robot>

Commit message: Henk

File: src/assignment4/urdf/lynxmotion.urdf.xacro (robot description, xacro)
@@ -1,4 +1,4 @@
 <?xml version="1.0"?>
-<robot name="macroed" xmlns:xacro="http://ros.org/wiki/xacro">
+<robot name="Swekbot 1.33.7" xmlns:xacro="http://ros.org/wiki/xacro">
   <xacro:property name="M_PI" value="3.14159"/>
   <xacro:property name="base_width" value="0.069" />
@@ -8,6 +8,8 @@
   <xacro:property name="shoulder_height" value="0.010" />
   <xacro:property name="shoulder_offset" value="0.015" />
-  <xacro:property name="upperarm_length" value="0.127" />
-  <xacro:property name="hand_length" value="0.086" />
+  <xacro:property name="upperarm_length" value="0.121" />
+  <xacro:property name="lowerarm_length" value="0.127" />
+  <xacro:property name="gripper_length" value="0.086" />
+  <xacro:property name="gripper_size" value="0.015" />
   <!-- Links -->
   <link name="base_link">
@@ -43,5 +45,5 @@
     </visual>
   </link>
-  <!-- <link name="elbow_link">
+  <link name="elbow_link">
     <visual>
       <origin xyz="0 0 0" rpy="0 0 0"/>
@@ -50,5 +52,37 @@
       </geometry>
     </visual>
-  </link> -->
+  </link>
+  <link name="lowerarm_link">
+    <visual>
+      <origin xyz="0 0 0" rpy="0 0 0"/>
+      <geometry>
+        <box size="${lowerarm_length} ${servo_width} ${servo_width}"/>
+      </geometry>
+    </visual>
+  </link>
+  <link name="wrist_link">
+    <visual>
+      <origin xyz="0 0 0" rpy="0 0 0"/>
+      <geometry>
+        <cylinder radius="${servo_width}" length="${servo_length}"/>
+      </geometry>
+    </visual>
+  </link>
+  <link name="gripper_left">
+    <visual>
+      <origin xyz="0 0 0" rpy="0 0 0"/>
+      <geometry>
+        <box size="${gripper_length} ${gripper_size} ${gripper_size}"/>
+      </geometry>
+    </visual>
+  </link>
+  <link name="gripper_right">
+    <visual>
+      <origin xyz="0 0 0" rpy="0 0 0"/>
+      <geometry>
+        <box size="${gripper_length} ${gripper_size} ${gripper_size}"/>
+      </geometry>
+    </visual>
+  </link>
   <!-- Joints -->
   <joint name="shoulder_rotate_joint" type="revolute">
@@ -71,10 +105,36 @@
     <child link="upperarm_link"/>
   </joint>
-  <!-- <joint name="elbow_joint" type="revolute">
-    <origin xyz="0 0 0" rpy="${M_PI/2} 0 0"/>
+  <joint name="elbow_joint" type="revolute">
+    <origin xyz="${upperarm_length/2} 0 0" rpy="${M_PI/2} 0 0"/>
     <parent link="upperarm_link"/>
     <child link="elbow_link"/>
     <axis xyz="0 0 1"/>
     <limit lower="-${M_PI/2}" upper="${M_PI/2}" effort="0" velocity="3.67"/>
-  </joint> -->
+  </joint>
+  <joint name="lowerarm_joint" type="fixed">
+    <origin xyz="${lowerarm_length/2} 0 0" rpy="${M_PI/2} 0 0"/>
+    <parent link="elbow_link"/>
+    <child link="lowerarm_link"/>
+  </joint>
+  <joint name="wrist_joint" type="revolute">
+    <origin xyz="${upperarm_length/2} 0 0" rpy="${M_PI/2} 0 0"/>
+    <parent link="lowerarm_link"/>
+    <child link="wrist_link"/>
+    <axis xyz="0 0 1"/>
+    <limit lower="-${M_PI/2}" upper="${M_PI/2}" effort="0" velocity="3.67"/>
+  </joint>
+  <joint name="gripper_left_joint" type="planar">
+    <origin xyz="${upperarm_length/2} 0 0" rpy="${M_PI/2} 0 0"/>
+    <parent link="wrist_link"/>
+    <child link="gripper_left"/>
+    <axis xyz="0 0 1"/>
+    <limit lower="-${M_PI/2}" upper="${M_PI/2}" effort="0" velocity="3.67"/>
+  </joint>
+  <joint name="gripper_right_joint" type="planar">
+    <origin xyz="${upperarm_length/2} 0 0" rpy="${M_PI/2} 0 0"/>
+    <parent link="wrist_link"/>
+    <child link="gripper_right"/>
+    <axis xyz="0 0 1"/>
+    <limit lower="-${M_PI/2}" upper="${M_PI/2}" effort="0" velocity="3.67"/>
+  </joint>
 </robot>

Commit message: Thing is done

File: src/assignment4/urdf/lynxmotion.urdf.xacro (robot description, xacro)
@@ -12,4 +12,5 @@
   <xacro:property name="gripper_length" value="0.086" />
   <xacro:property name="gripper_size" value="0.015" />
+  <xacro:property name="gripper_open" value="0.10" />
   <!-- Links -->
   <link name="base_link">
@@ -69,5 +70,13 @@
     </visual>
   </link>
-  <link name="gripper_left">
+  <link name="gripper_base_link">
+    <visual>
+      <origin xyz="0 0 0" rpy="0 0 0"/>
+      <geometry>
+        <box size="${gripper_size} ${gripper_open+gripper_size*2} ${gripper_size}"/>
+      </geometry>
+    </visual>
+  </link>
+  <link name="gripper_left_link">
     <visual>
       <origin xyz="0 0 0" rpy="0 0 0"/>
@@ -77,5 +86,5 @@
     </visual>
   </link>
-  <link name="gripper_right">
+  <link name="gripper_right_link">
     <visual>
       <origin xyz="0 0 0" rpy="0 0 0"/>
@@ -124,17 +133,22 @@
     <limit lower="-${M_PI/2}" upper="${M_PI/2}" effort="0" velocity="3.67"/>
   </joint>
-  <joint name="gripper_left_joint" type="planar">
-    <origin xyz="${upperarm_length/2} 0 0" rpy="${M_PI/2} 0 0"/>
+  <joint name="gripper_base_joint" type="fixed">
+    <origin xyz="${servo_width} 0 0" rpy="0 0 0"/>
     <parent link="wrist_link"/>
-    <child link="gripper_left"/>
+    <child link="gripper_base_link"/>
+  </joint>
+  <joint name="gripper_left_joint" type="prismatic">
+    <origin xyz="${gripper_length/2} ${gripper_size/2} 0" rpy="${M_PI/2} 0 0"/>
+    <parent link="gripper_base_link"/>
+    <child link="gripper_left_link"/>
     <axis xyz="0 0 1"/>
-    <limit lower="-${M_PI/2}" upper="${M_PI/2}" effort="0" velocity="3.67"/>
+    <limit lower="-${gripper_open/2}" upper="0" effort="0" velocity="3.67"/>
   </joint>
-  <joint name="gripper_right_joint" type="planar">
-    <origin xyz="${upperarm_length/2} 0 0" rpy="${M_PI/2} 0 0"/>
-    <parent link="wrist_link"/>
-    <child link="gripper_right"/>
+  <joint name="gripper_right_joint" type="prismatic">
+    <origin xyz="${gripper_length/2} -${gripper_size/2} 0" rpy="${M_PI/2} 0 0"/>
+    <parent link="gripper_base_link"/>
+    <child link="gripper_right_link"/>
     <axis xyz="0 0 1"/>
-    <limit lower="-${M_PI/2}" upper="${M_PI/2}" effort="0" velocity="3.67"/>
+    <limit lower="0" upper="${gripper_open/2}" effort="0" velocity="3.67"/>
   </joint>
 </robot>
